File: Hardware/CSS811_CO2_TVOC_Breakout.brd (EAGLE design)
At the start: 17.8 x 17.8 mm, 20 parts, among them U2 CCS811

Commit message: Updated to take care of checklist and review items
Parts:
- U2: device CCS811_Breakout_Temp:LGA10-2.7X4.0MM -> CCS811_Breakout_Temp:LGA10
- moved FD1 4.07 mm to (4.83, 16.9)
- moved FD2 1.27 mm to (15.2, 3.81)
Other:
- board text added: "All measurements in inches"
Changed lines of the file:
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@@
 <setting verticaltext="up"/>
 </settings>
-<grid distance="0.05" unitdist="inch" unit="inch" style="lines" multiple="1" display="yes" altdistance="0.005" altunitdist="inch" altunit="inch"/>
+<grid distance="0.05" unitdist="inch" unit="inch" style="lines" multiple="1" display="yes" altdistance="0.001" altunitdist="inch" altunit="inch"/>
 <layers>
-<layer number="1" name="Top" color="4" fill="1" visible="no" active="yes"/>
+<layer number="1" name="Top" color="4" fill="1" visible="yes" active="yes"/>
 <layer number="2" name="Route2" color="1" fill="3" visible="no" active="no"/>
 <layer number="3" name="Route3" color="4" fill="3" visible="no" active="no"/>
@@
 <layer number="19" name="Unrouted" color="6" fill="1" visible="yes" active="yes"/>
 <layer number="20" name="Dimension" color="15" fill="1" visible="yes" active="yes"/>
-<layer number="21" name="tPlace" color="16" fill="1" visible="no" active="yes"/>
+<layer number="21" name="tPlace" color="16" fill="1" visible="yes" active="yes"/>
 <layer number="22" name="bPlace" color="14" fill="1" visible="yes" active="yes"/>
 <layer number="23" name="tOrigins" color="15" fill="1" visible="no" active="yes"/>
-<layer number="24" name="bOrigins" color="15" fill="1" visible="yes" active="yes"/>
+<layer number="24" name="bOrigins" color="15" fill="1" visible="no" active="yes"/>
 <layer number="25" name="tNames" color="7" fill="1" visible="no" active="yes"/>
 <layer number="26" name="bNames" color="7" fill="1" visible="no" active="yes"/>
 <layer number="27" name="tValues" color="7" fill="1" visible="no" active="yes"/>
 <layer number="28" name="bValues" color="7" fill="1" visible="no" active="yes"/>
-<layer number="29" name="tStop" color="7" fill="3" visible="no" active="yes"/>
+<layer number="29" name="tStop" color="7" fill="3" visible="yes" active="yes"/>
 <layer number="30" name="bStop" color="7" fill="6" visible="no" active="yes"/>
-<layer number="31" name="tCream" color="7" fill="4" visible="no" active="yes"/>
+<layer number="31" name="tCream" color="7" fill="4" visible="yes" active="yes"/>
 <layer number="32" name="bCream" color="7" fill="5" visible="no" active="yes"/>
 <layer number="33" name="tFinish" color="6" fill="3" visible="no" active="yes"/>
@@
 <layer number="37" name="tTest" color="7" fill="1" visible="no" active="yes"/>
 <layer number="38" name="bTest" color="7" fill="1" visible="no" active="yes"/>
-<layer number="39" name="tKeepout" color="4" fill="11" visible="no" active="yes"/>
+<layer number="39" name="tKeepout" color="4" fill="11" visible="yes" active="yes"/>
 <layer number="40" name="bKeepout" color="1" fill="11" visible="no" active="yes"/>
 <layer number="41" name="tRestrict" color="4" fill="10" visible="no" active="yes"/>
@@
 <layer number="45" name="Holes" color="7" fill="1" visible="no" active="yes"/>
 <layer number="46" name="Milling" color="3" fill="1" visible="no" active="yes"/>
-<layer number="47" name="Measures" color="7" fill="1" visible="no" active="yes"/>
+<layer number="47" name="Measures" color="7" fill="1" visible="yes" active="yes"/>
 <layer number="48" name="Document" color="7" fill="1" visible="no" active="yes"/>
 <layer number="49" name="Reference" color="7" fill="1" visible="no" active="yes"/>
@@
 <text x="13.97" y="2.794" size="1.016" layer="22" font="vector" ratio="15" rot="MR90" align="center-left">3.3V</text>
 <text x="16.51" y="2.794" size="1.016" layer="22" font="vector" ratio="15" rot="MR90" align="center-left">GND</text>
-<text x="9.017" y="16.51" size="1.2065" layer="21" ratio="15" align="center">CCS811</text>
+<text x="9.017" y="16.51" size="1.2065" layer="21" font="vector" ratio="15" align="center">CCS811</text>
 <text x="17.399" y="10.287" size="1.016" layer="16" ratio="20" rot="SMR270" align="bottom-center">v10</text>
-<text x="4.191" y="10.287" size="0.889" layer="22" ratio="15" rot="MR90" align="bottom-center">ADDR</text>
+<text x="4.191" y="10.287" size="0.889" layer="22" font="vector" ratio="15" rot="MR90" align="bottom-center">ADDR</text>
 <text x="16.51" y="-21.59" size="1.778" layer="51">Nathan Seidle</text>
-<text x="17.399" y="10.287" size="1.016" layer="21" ratio="15" rot="R90" align="bottom-center">NTC</text>
-<text x="9.017" y="14.859" size="1.016" layer="21" ratio="15" align="center">Air Quality</text>
-<text x="0.381" y="10.287" size="0.889" layer="22" ratio="15" rot="MR90" align="bottom-center">I2C PU</text>
+<text x="17.399" y="10.287" size="1.016" layer="21" font="vector" ratio="15" rot="R90" align="bottom-center">NTC</text>
+<text x="9.017" y="14.859" size="1.016" layer="21" font="vector" ratio="15" align="center">Air Quality</text>
+<text x="0.381" y="10.287" size="0.889" layer="22" font="vector" ratio="15" rot="MR90" align="bottom-center">I2C PU</text>
 <text x="6.35" y="2.794" size="1.016" layer="21" font="vector" ratio="15" rot="R90" align="center-left">!WAK</text>
 <text x="3.81" y="2.794" size="1.016" layer="21" font="vector" ratio="15" rot="R90" align="center-left">!INT</text>
@@
 <text x="3.81" y="2.794" size="1.016" layer="22" font="vector" ratio="15" rot="MR90" align="center-left">!INT</text>
 <text x="1.27" y="2.794" size="1.016" layer="22" font="vector" ratio="15" rot="MR90" align="center-left">!RST</text>
+<dimension x1="2.54" y1="15.24" x2="0" y2="0" x3="-2.54" y3="7.62" textsize="1.778" layer="47" dtype="vertical" unit="inch"/>
+<dimension x1="0" y1="17.78" x2="0" y2="0" x3="-6.35" y3="8.89" textsize="1.778" layer="47" dtype="vertical" unit="inch"/>
+<dimension x1="2.54" y1="15.24" x2="0" y2="15.24" x3="1.27" y3="20.32" textsize="1.778" layer="47" dtype="horizontal" unit="inch"/>
+<dimension x1="15.24" y1="15.24" x2="0" y2="15.24" x3="7.62" y3="24.13" textsize="1.778" layer="47" dtype="horizontal" unit="inch"/>
+<dimension x1="17.78" y1="17.78" x2="0" y2="17.78" x3="8.89" y3="27.94" textsize="1.778" layer="47" dtype="horizontal" unit="inch"/>
+<text x="24.13" y="22.86" size="1.778" layer="47">All measurements in inches</text>
 </plain>
 <attributes>
@@
 </element>
 <element name="LOGO4" library="SparkFun-Aesthetics" package="OSHW-LOGO-S" value="OSHW-LOGOS" x="8.89" y="7.62" rot="MR0"/>
-<element name="FD1" library="SparkFun-Aesthetics" package="FIDUCIAL-1X2" value="FIDUCIAL1X2" x="0.762" y="17.018"/>
-<element name="FD2" library="SparkFun-Aesthetics" package="FIDUCIAL-1X2" value="FIDUCIAL1X2" x="15.24" y="2.54"/>
+<element name="FD1" library="SparkFun-Aesthetics" package="FIDUCIAL-1X2" value="FIDUCIAL1X2" x="4.826" y="16.891"/>
+<element name="FD2" library="SparkFun-Aesthetics" package="FIDUCIAL-1X2" value="FIDUCIAL1X2" x="15.24" y="3.81"/>
 <element name="R2" library="SparkFun-Resistors" package="0603" value="4.7k" x="6.985" y="6.35" rot="R180">
 <attribute name="PROD_ID" value="RES-07857" x="6.985" y="6.35" size="1.778" layer="27" font="vector" ratio="15" rot="R180" display="off"/>
 </element>
 <element name="J2" library="SparkFun-Connectors" package="1X03_NO_SILK" value="" x="6.35" y="1.27" rot="R180"/>
-<element name="U2" library="CCS811_Breakout_Temp" package="LGA10-2.7X4.0MM" value="CCS811" x="8.89" y="10.16" rot="R90">
+<element name="U2" library="CCS811_Breakout_Temp" package="LGA10" value="CCS811" x="8.89" y="10.16" rot="R90">
 <attribute name="PROD_ID" value="IC-13607" x="8.89" y="10.16" size="1.778" layer="27" rot="R90" display="off"/>
+<attribute name="VALUE" value="CCS811" x="8.89" y="10.16" size="1.778" layer="27" rot="R90" display="off"/>
 </element>
 <element name="R1" library="SparkFun-Resistors" package="0603" value="100k" x="10.795" y="6.35" rot="R180">
