File: Hardware/CSS811_CO2_TVOC_Breakout.sch (EAGLE design)
At the start: 20 parts, among them U2 CCS811

Commit message: Updated to take care of checklist and review items
Changed lines of the file:
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@@
 <instance part="R2" gate="G$1" x="55.88" y="139.7" rot="R90"/>
 <instance part="J2" gate="J$1" x="106.68" y="48.26" rot="R180"/>
-<instance part="U2" gate="G$1" x="78.74" y="129.54"/>
+<instance part="U2" gate="U1" x="78.74" y="129.54"/>
 <instance part="R1" gate="G$1" x="96.52" y="38.1" rot="R90"/>
 <instance part="GND1" gate="1" x="96.52" y="27.94" rot="MR0"/>
@@
 <wire x1="66.04" y1="119.38" x2="63.5" y2="119.38" width="0.1524" layer="91"/>
 <wire x1="63.5" y1="119.38" x2="63.5" y2="116.84" width="0.1524" layer="91"/>
-<pinref part="U2" gate="G$1" pin="GND"/>
+<pinref part="U2" gate="U1" pin="GND"/>
 </segment>
 <segment>
@@
 <wire x1="91.44" y1="134.62" x2="93.98" y2="134.62" width="0.1524" layer="91"/>
 <label x="93.98" y="134.62" size="1.27" layer="95" font="vector" xref="yes"/>
-<pinref part="U2" gate="G$1" pin="SCL"/>
+<pinref part="U2" gate="U1" pin="SCL"/>
 </segment>
 <segment>
@@
 <wire x1="91.44" y1="137.16" x2="93.98" y2="137.16" width="0.1524" layer="91"/>
 <label x="93.98" y="137.16" size="1.27" layer="95" font="vector" xref="yes"/>
-<pinref part="U2" gate="G$1" pin="SDA"/>
+<pinref part="U2" gate="U1" pin="SDA"/>
 </segment>
 <segment>
@@
 <pinref part="SUPPLY3" gate="G$1" pin="3.3V"/>
 <wire x1="63.5" y1="137.16" x2="63.5" y2="147.32" width="0.1524" layer="91"/>
-<pinref part="U2" gate="G$1" pin="VDD"/>
+<pinref part="U2" gate="U1" pin="VDD"/>
 </segment>
 <segment>
@@
 <label x="53.34" y="132.08" size="1.27" layer="95" font="vector" rot="R180" xref="yes"/>
 <pinref part="R2" gate="G$1" pin="1"/>
-<pinref part="U2" gate="G$1" pin="!RESET!"/>
+<pinref part="U2" gate="U1" pin="!RESET!"/>
 </segment>
 <segment>
@@
 <wire x1="106.68" y1="116.84" x2="106.68" y2="119.38" width="0.1524" layer="91"/>
 <junction x="106.68" y="119.38"/>
-<pinref part="U2" gate="G$1" pin="ADDR"/>
+<pinref part="U2" gate="U1" pin="ADDR"/>
 </segment>
 </net>
@@
 <wire x1="91.44" y1="124.46" x2="93.98" y2="124.46" width="0.1524" layer="91"/>
 <label x="93.98" y="124.46" size="1.27" layer="95" font="vector" xref="yes"/>
-<pinref part="U2" gate="G$1" pin="AUX"/>
+<pinref part="U2" gate="U1" pin="AUX"/>
 </segment>
 <segment>
@@
 <wire x1="91.44" y1="129.54" x2="93.98" y2="129.54" width="0.1524" layer="91"/>
 <label x="93.98" y="129.54" size="1.27" layer="95" font="vector" xref="yes"/>
-<pinref part="U2" gate="G$1" pin="!INT!"/>
+<pinref part="U2" gate="U1" pin="!INT!"/>
 </segment>
 <segment>
@@
 <wire x1="91.44" y1="132.08" x2="93.98" y2="132.08" width="0.1524" layer="91"/>
 <label x="93.98" y="132.08" size="1.27" layer="95" font="vector" xref="yes"/>
-<pinref part="U2" gate="G$1" pin="!WAKE!"/>
+<pinref part="U2" gate="U1" pin="!WAKE!"/>
 </segment>
 <segment>
@@
 <junction x="63.5" y="127"/>
 <label x="58.42" y="127" size="1.27" layer="95" font="vector" rot="R180" xref="yes"/>
-<pinref part="U2" gate="G$1" pin="PWM"/>
-<pinref part="U2" gate="G$1" pin="SENSE"/>
+<pinref part="U2" gate="U1" pin="PWM"/>
+<pinref part="U2" gate="U1" pin="SENSE"/>
 </segment>
 <segment>
@@
 </sheet>
 </sheets>
+<errors>
+</errors>
 </schematic>
 </drawing>
